File: ControlBoardMain.sch (EAGLE design)
At the start: 11 parts, among them J1 350759-4, J2 RPI_HEADER, J3 DC_POWERJACK, J4 22-23-2021, Q1 NMOS, U1 VOLTAGE_REGULATOR

Commit message: Added flyback diode
Parts:
- added D1: DIODE, 00_ThruHole:DIODE
Connections:
- net GND: now also D1.P2
- net PUMP_GND: now also D1.P1
Changed lines of the file:
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@@
 <part name="J4" library="con-molex" deviceset="22-23-2021" device=""/>
 <part name="U$1" library="1111Lib" deviceset="LOGO" device=""/>
+<part name="D1" library="00_ThruHole" deviceset="DIODE" device=""/>
 </parts>
 <sheets>
@@
 <instance part="J4" gate="-2" x="99.06" y="205.74"/>
 <instance part="U$1" gate="G$1" x="375.92" y="5.08"/>
+<instance part="D1" gate="D$1" x="78.74" y="139.7" rot="R180"/>
 </instances>
 <busses>
@@
 <pinref part="SUPPLY2" gate="GND" pin="GND"/>
 <wire x1="63.5" y1="119.126" x2="63.5" y2="116.84" width="0.1524" layer="91"/>
+<pinref part="D1" gate="D$1" pin="P2"/>
+<wire x1="78.74" y1="121.92" x2="78.74" y2="119.126" width="0.1524" layer="91"/>
+<wire x1="78.74" y1="119.126" x2="63.5" y2="119.126" width="0.1524" layer="91"/>
+<junction x="63.5" y="119.126"/>
 </segment>
 <segment>
@@
 <pinref part="Q1" gate="Q$1" pin="DRAIN"/>
 <wire x1="48.26" y1="147.32" x2="63.5" y2="147.32" width="0.1524" layer="91"/>
-<wire x1="63.5" y1="147.32" x2="63.5" y2="142.24" width="0.1524" layer="91"/>
+<wire x1="63.5" y1="147.32" x2="63.5" y2="144.78" width="0.1524" layer="91"/>
 <pinref part="J1" gate="G$1" pin="1"/>
+<wire x1="63.5" y1="144.78" x2="63.5" y2="142.24" width="0.1524" layer="91"/>
 <wire x1="76.2" y1="154.94" x2="76.2" y2="147.32" width="0.1524" layer="91"/>
 <wire x1="76.2" y1="147.32" x2="63.5" y2="147.32" width="0.1524" layer="91"/>
 <junction x="63.5" y="147.32"/>
+<pinref part="D1" gate="D$1" pin="P1"/>
+<wire x1="78.74" y1="139.7" x2="78.74" y2="144.78" width="0.1524" layer="91"/>
+<wire x1="78.74" y1="144.78" x2="63.5" y2="144.78" width="0.1524" layer="91"/>
+<junction x="63.5" y="144.78"/>
 </segment>
 </net>

Commit message: Fixed the flyback diode
Connections:
- net GND: no longer D1.P2
- net PUMP_GND: now also D1.P2; no longer D1.P1
- net VIN: now also D1.P1
Other:
- moved on the sheet: D1
Changed lines of the file:
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@@
 <text x="73.66" y="162.56" size="2.54" layer="150">Pump Header</text>
 <text x="40.64" y="215.9" size="2.54" layer="150">RPi Voltage Regulator</text>
-<text x="83.82" y="132.08" size="1.778" layer="150">This low side driver controls the pump.
+<text x="88.9" y="121.92" size="1.778" layer="150">This low side driver controls the pump.
 R2 pulls the pump high to Vin (12V).
 Pump_On is held low until pulled high
@@
 <instance part="J4" gate="-2" x="99.06" y="205.74"/>
 <instance part="U$1" gate="G$1" x="375.92" y="5.08"/>
-<instance part="D1" gate="D$1" x="78.74" y="139.7" rot="R180"/>
+<instance part="D1" gate="D$1" x="88.9" y="137.16" rot="R90"/>
 </instances>
 <busses>
@@
 <pinref part="SUPPLY2" gate="GND" pin="GND"/>
 <wire x1="63.5" y1="119.126" x2="63.5" y2="116.84" width="0.1524" layer="91"/>
-<pinref part="D1" gate="D$1" pin="P2"/>
-<wire x1="78.74" y1="121.92" x2="78.74" y2="119.126" width="0.1524" layer="91"/>
-<wire x1="78.74" y1="119.126" x2="63.5" y2="119.126" width="0.1524" layer="91"/>
-<junction x="63.5" y="119.126"/>
 </segment>
 <segment>
@@
 <pinref part="Q1" gate="Q$1" pin="DRAIN"/>
 <wire x1="48.26" y1="147.32" x2="63.5" y2="147.32" width="0.1524" layer="91"/>
-<wire x1="63.5" y1="147.32" x2="63.5" y2="144.78" width="0.1524" layer="91"/>
 <pinref part="J1" gate="G$1" pin="1"/>
-<wire x1="63.5" y1="144.78" x2="63.5" y2="142.24" width="0.1524" layer="91"/>
+<wire x1="63.5" y1="147.32" x2="63.5" y2="142.24" width="0.1524" layer="91"/>
 <wire x1="76.2" y1="154.94" x2="76.2" y2="147.32" width="0.1524" layer="91"/>
-<wire x1="76.2" y1="147.32" x2="63.5" y2="147.32" width="0.1524" layer="91"/>
+<wire x1="76.2" y1="147.32" x2="71.12" y2="147.32" width="0.1524" layer="91"/>
 <junction x="63.5" y="147.32"/>
-<pinref part="D1" gate="D$1" pin="P1"/>
-<wire x1="78.74" y1="139.7" x2="78.74" y2="144.78" width="0.1524" layer="91"/>
-<wire x1="78.74" y1="144.78" x2="63.5" y2="144.78" width="0.1524" layer="91"/>
-<junction x="63.5" y="144.78"/>
+<pinref part="D1" gate="D$1" pin="P2"/>
+<wire x1="71.12" y1="147.32" x2="63.5" y2="147.32" width="0.1524" layer="91"/>
+<wire x1="71.12" y1="137.16" x2="71.12" y2="147.32" width="0.1524" layer="91"/>
+<junction x="71.12" y="147.32"/>
 </segment>
 </net>
@@
 <pinref part="J1" gate="G$1" pin="2"/>
 <wire x1="78.74" y1="154.94" x2="78.74" y2="147.32" width="0.1524" layer="91"/>
-<wire x1="78.74" y1="147.32" x2="93.98" y2="147.32" width="0.1524" layer="91"/>
+<wire x1="78.74" y1="147.32" x2="88.9" y2="147.32" width="0.1524" layer="91"/>
 <label x="88.9" y="147.32" size="2.54" layer="95"/>
+<pinref part="D1" gate="D$1" pin="P1"/>
+<wire x1="88.9" y1="147.32" x2="93.98" y2="147.32" width="0.1524" layer="91"/>
+<wire x1="88.9" y1="137.16" x2="88.9" y2="147.32" width="0.1524" layer="91"/>
+<junction x="88.9" y="147.32"/>
 </segment>
 </net>
